File: PCB/KiCad file.kicad_pcb (KiCad board)
At the start: 2 copper layers, 90.3 x 79.8 mm, 25 parts, among them SW1 SW_Push, SW10 SW_Push, SW13 RotaryEncoder_Switch, SW14 RotaryEncoder_Switch, SW2 SW_Push, SW3 SW_Push, SW4 SW_Push, SW5 SW_Push, SW6 SW_Push, SW7 SW_Push, SW8 SW_Push, SW9 SW_Push, U1 MOUDLE-SEEEDUINO-XIAO, U2 PCF8574AT

Commit message: Made the hackpad and changed everything so it is better. Added pull up resistors and madee code actually work
Parts:
- added R1: 4.7k, Resistor_SMD:R_0805_2012Metric, B.Cu at (174.9, 48.6)
- added R2: 4.7k, Resistor_SMD:R_0805_2012Metric, B.Cu at (174.9, 51.6)
Routing:
- net SDA: track 28.4 -> 71.7 mm
- net 3V3: track 55.7 -> 82.9 mm
- net SCL: track 28.6 -> 55.2 mm
