File: PCB/KiCad file.kicad_sch (KiCad schematic)
At the start: 25 parts, among them SW1 SW_Push, SW10 SW_Push, SW13 RotaryEncoder_Switch, SW14 RotaryEncoder_Switch, SW2 SW_Push, SW3 SW_Push, SW4 SW_Push, SW5 SW_Push, SW6 SW_Push, SW7 SW_Push, SW8 SW_Push, SW9 SW_Push, U1 MOUDLE-SEEEDUINO-XIAO, U2 PCF8574AT

Commit message: Added many changes, most minor but some major.
I created my readme and added an assets folder to load screenshots into the readme. Also, I added PCB libraries so others can make their own version of the PCB.
Connections:
- no-connect marks 0 -> 4
Changed lines of the file:
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@@
 	)
 	(junction
+		(at 77.47 43.18)
+		(diameter 0)
+		(color 0 0 0 0)
+	)
+	(junction
 		(at 152.4 63.5)
 		(diameter 0)
 		(color 0 0 0 0)
 	)
+	(no_connect
+		(at 77.47 48.26)
+	)
+	(no_connect
+		(at 77.47 38.1)
+	)
+	(no_connect
+		(at 64.77 157.48)
+	)
+	(no_connect
+		(at 77.47 45.72)
+	)
 	(wire
 		(pts
@@
 	(wire
 		(pts
+			(xy 81.28 45.72) (xy 77.47 43.18)
+		)
+		(stroke
+			(width 0)
+			(type default)
+		)
+	)
+	(wire
+		(pts
 			(xy 30.48 134.62) (xy 54.61 134.62)
 		)
@@
 	(global_label "3V3"
 		(shape output)
-		(at 77.47 43.18 0)
+		(at 81.28 45.72 0)
 		(fields_autoplaced yes)
 		(effects
@@
 		)
 		(property "Intersheetrefs" "${INTERSHEET_REFS}"
-			(at 83.9628 43.18 0)
+			(at 87.7728 45.72 0)
 			(hide yes)
 			(show_name no)
@@
 	(symbol
 		(lib_id "power:GND")
-		(at 25.4 162.56 0)
+		(at 25.4 162.56 270)
 		(unit 1)
 		(body_style 1)
@@
 		(fields_autoplaced yes)
 		(property "Reference" "#PWR02"
-			(at 25.4 168.91 0)
+			(at 19.05 162.56 0)
 			(hide yes)
 			(show_name no)
@@
 		)
 		(property "Value" "GND"
-			(at 25.4 167.64 0)
+			(at 24.13 158.75 90)
 			(show_name no)
 			(do_not_autoplace no)
@@
 	)
 	(symbol
+		(lib_id "power:PWR_FLAG")
+		(at 30.48 162.56 180)
+		(unit 1)
+		(body_style 1)
+		(exclude_from_sim no)
+		(in_bom yes)
+		(on_board yes)
+		(in_pos_files yes)
+		(dnp no)
+		(fields_autoplaced yes)
+		(property "Reference" "#FLG02"
+			(at 30.48 164.465 0)
+			(hide yes)
+			(show_name no)
+			(do_not_autoplace no)
+			(effects
+				(font
+					(size 1.27 1.27)
+				)
+			)
+		)
+		(property "Value" "PWR_FLAG"
+			(at 30.48 167.64 0)
+			(show_name no)
+			(do_not_autoplace no)
+			(effects
+				(font
+					(size 1.27 1.27)
+				)
+			)
+		)
+		(property "Footprint" ""
+			(at 30.48 162.56 0)
+			(hide yes)
+			(show_name no)
+			(do_not_autoplace no)
+			(effects
+				(font
+					(size 1.27 1.27)
+				)
+			)
+		)
+		(property "Datasheet" ""
+			(at 30.48 162.56 0)
+			(hide yes)
+			(show_name no)
+			(do_not_autoplace no)
+			(effects
+				(font
+					(size 1.27 1.27)
+				)
+			)
+		)
+		(property "Description" "Special symbol for telling ERC where power comes from"
+			(at 30.48 162.56 0)
+			(hide yes)
+			(show_name no)
+			(do_not_autoplace no)
+			(effects
+				(font
+					(size 1.27 1.27)
+				)
+			)
+		)
+		(pin "1"
+		)
+		(instances
+			(project "KiCad file"
+				(path "/03a2f365-6f86-40de-8236-abbe5f4614e3"
+					(reference "#FLG02")
+					(unit 1)
+				)
+			)
+		)
+	)
+	(symbol
 		(lib_id "Switch:SW_Push")
 		(at 208.28 63.5 0)
@@
 					(unit 1)
 				)
+			)
+		)
+	)
+	(symbol
+		(lib_id "power:PWR_FLAG")
+		(at 77.47 43.18 270)
+		(unit 1)
+		(body_style 1)
+		(exclude_from_sim no)
+		(in_bom yes)
+		(on_board yes)
+		(in_pos_files yes)
+		(dnp no)
+		(fields_autoplaced yes)
+		(property "Reference" "#FLG01"
+			(at 79.375 43.18 0)
+			(hide yes)
+			(show_name no)
+			(do_not_autoplace no)
+			(effects
+				(font
+					(size 1.27 1.27)
+				)
+			)
+		)
+		(property "Value" "PWR_FLAG"
+			(at 81.28 43.1799 90)
+			(show_name no)
+			(do_not_autoplace no)
+			(effects
+				(font
+					(size 1.27 1.27)
+				)
+				(justify left)
+			)
+		)
+		(property "Footprint" ""
+			(at 77.47 43.18 0)
+			(hide yes)
+			(show_name no)
+			(do_not_autoplace no)
+			(effects
+				(font
+					(size 1.27 1.27)
+				)
+			)
+		)
+		(property "Datasheet" ""
+			(at 77.47 43.18 0)
+			(hide yes)
+			(show_name no)
+			(do_not_autoplace no)
+			(effects
+				(font
+					(size 1.27 1.27)
+				)
+			)
+		)
+		(property "Description" "Special symbol for telling ERC where power comes from"
+			(at 77.47 43.18 0)
+			(hide yes)
+			(show_name no)
+			(do_not_autoplace no)
+			(effects
+				(font
+					(size 1.27 1.27)
+				)
+			)
+		)
+		(pin "1"
+		)
+		(instances
+			(project "KiCad file"
+				(path "/03a2f365-6f86-40de-8236-abbe5f4614e3"
+					(reference "#FLG01")
+					(unit 1)
+				)

Commit message: Made the hackpad and changed everything so it is better. Added pull up resistors and madee code actually work
Parts:
- added R1, R2: 4.7k, Resistor_SMD:R_0805_2012Metric, symbol Device:R
- C1: LCSC Part # (none) -> C49678
- D1, D10, D2, D3, D4, D5, D6, D7, D8, D9: LCSC Part # (none) -> C85057
- SW1, SW10, SW2, SW3, SW4, SW5, SW6, SW7, SW8, SW9: JLCPCB Part # (none) -> C9900177322
- U2: LCSC Part # (none) -> C86832
Connections:
- net 3V3: now also R1.1, R2.1
- net SCL: now also R2.2
- net SDA: now also R1.2
